File: clock-module--100mmX100mm.kicad_pcb (KiCad board)
At the start: 2 copper layers, 56 x 100 mm, 35 parts, among them P1 CONN_01X01, P2 CONN_01X01, P3 CONN_01X01, P4 CONN_01X01, P5 CONN_01X01, P6 CONN_01X01, P7 CONN_01X01, P8 CONN_01X01, SW1 SW_SPDT, SW2 SW_SPST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

Commit message: Improve pad clearences, aligator clip improvements
Routing:
- net GND: track 13.5 -> 26.0 mm
- net +5V: track 267.1 -> 271.1 mm
- net Net-(R4-Pad2): track 41.1 -> 42.8 mm
Other:
- rule pad_to_mask_clearance: 0.5 -> 0.2

Commit message: Fix bug in board layout
Connections:
- R8 pad 2: GND -> +5V
Routing:
- net +5V: track 271.1 -> 282.3 mm, vias 6 -> 8
Changed lines of the file:
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@@
     (links 73)
     (no_connects 0)
-    (area 57.435716 50.8 185.064286 167.700001)
+    (area 79.924999 59.924999 136.075001 160.075001)
     (thickness 1.6)
     (drawings 35)
-    (tracks 207)
+    (tracks 214)
     (zones 0)
     (modules 35)
@@
     (visible_elements FFFFFFFF)
     (pcbplotparams
-      (layerselection 0x01020_80000001)
+      (layerselection 0x010e0_80000001)
       (usegerberextensions true)
       (excludeedgelayer true)
@@
       (net 26 "Net-(R8-Pad1)"))
     (pad 2 thru_hole oval (at 10.16 0) (size 1.6 1.6) (drill 0.8) (layers *.Cu *.Mask)
-      (net 18 GND))
+      (net 2 +5V))
     (model Resistors_THT.3dshapes/R_Axial_DIN0207_L6.3mm_D2.5mm_P10.16mm_Horizontal.wrl
       (at (xyz 0 0 0))
@@
   (segment (start 109.84 81) (end 103.54 81) (width 0.1524) (layer F.Cu) (net 1))
   (segment (start 103.54 81) (end 102 82.54) (width 0.1524) (layer F.Cu) (net 1))
+  (segment (start 120.91 113.75) (end 123.75 113.75) (width 0.1524) (layer F.Cu) (net 2))
+  (segment (start 123.75 113.75) (end 124 114) (width 0.1524) (layer F.Cu) (net 2))
+  (via (at 124 114) (size 0.6858) (drill 0.3302) (layers F.Cu B.Cu) (net 2))
+  (segment (start 124 108) (end 124 114) (width 0.1524) (layer B.Cu) (net 2))
+  (segment (start 124 106) (end 107 106) (width 0.3) (layer F.Cu) (net 2))
+  (segment (start 133 106) (end 124 106) (width 0.3) (layer F.Cu) (net 2))
+  (segment (start 124 106) (end 124 108) (width 0.1524) (layer F.Cu) (net 2))
+  (via (at 124 108) (size 0.6858) (drill 0.3302) (layers F.Cu B.Cu) (net 2))
   (segment (start 135.5 75) (end 135.5 99.576201) (width 0.3) (layer B.Cu) (net 2))
   (segment (start 128.5 73.5) (end 134 73.5) (width 0.3) (layer B.Cu) (net 2))
@@
   (segment (start 133 106) (end 134.576201 106) (width 0.3) (layer F.Cu) (net 2))
   (via (at 134.576201 106) (size 0.6858) (drill 0.3302) (layers F.Cu B.Cu) (net 2))
-  (segment (start 133 106) (end 107 106) (width 0.3) (layer F.Cu) (net 2))
   (segment (start 105 87) (end 96.3 87) (width 0.3) (layer F.Cu) (net 2))
   (segment (start 96.3 87) (end 94.38 85.08) (width 0.3) (layer F.Cu) (net 2))
@@
   (segment (start 98.76 106) (end 94.38 101.62) (width 0.3) (layer F.Cu) (net 2))
   (segment (start 105.92 106) (end 102 109.92) (width 0.3) (layer F.Cu) (net 2))
-  (segment (start 126.5 63.5) (end 128.5 65.5) (width 0.1524) (layer B.Cu) (net 2))
+  (segment (start 126.5 63.5) (end 128.5 65.5) (width 0.3) (layer B.Cu) (net 2))
   (segment (start 113 85.5) (end 111.623799 84.123799) (width 0.1524) (layer F.Cu) (net 3))
   (segment (start 111.623799 84.123799) (end 102.956201 84.123799) (width 0.1524) (layer F.Cu) (net 3))
@@
   (segment (start 109.21 132.21) (end 109.25 132.25) (width 0.1524) (layer F.Cu) (net 17))
   (via (at 109.25 132.25) (size 0.6858) (drill 0.3302) (layers F.Cu B.Cu) (net 17))
-  (segment (start 89.5 63.5) (end 89.5 64.914213) (width 0.1524) (layer B.Cu) (net 18))
-  (segment (start 89.5 64.914213) (end 89.5 76) (width 0.1524) (layer B.Cu) (net 18))
-  (segment (start 83.5 66) (end 87 66) (width 0.1524) (layer F.Cu) (net 18))
-  (segment (start 87 66) (end 89.5 63.5) (width 0.1524) (layer F.Cu) (net 18))
+  (segment (start 89.5 63.5) (end 89.5 64.914213) (width 0.3) (layer B.Cu) (net 18))
+  (segment (start 89.5 64.914213) (end 89.5 76) (width 0.3) (layer B.Cu) (net 18))
+  (segment (start 83.5 66) (end 87 66) (width 0.3) (layer F.Cu) (net 18))
+  (segment (start 87 66) (end 89.5 63.5) (width 0.3) (layer F.Cu) (net 18))
   (segment (start 133 98) (end 126.5 98) (width 0.1524) (layer F.Cu) (net 18))
   (segment (start 104 72) (end 104 63.5) (width 0.1524) (layer B.Cu) (net 19))
