File: clock-module.sch (KiCad schematic (older format))
At the start: 35 parts, among them P1 CONN_01X01, P2 CONN_01X01, P3 CONN_01X01, P4 CONN_01X01, P5 CONN_01X01, P6 CONN_01X01, P7 CONN_01X01, P8 CONN_01X01, SW1 SW_SPDT, SW2 SW_SPST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

Commit message: Fix bug in board layout
Connections:
- net +5V: now also R8.2
- net GND: no longer R8.2
Changed lines of the file:
@@
 	1    0    0    -1
-$EndComp
-$Comp
-L GND #PWR011
-U 1 1 589CFAE1
-P 2150 4450
-F 0 "#PWR011" H 2150 4200 50  0001 C CNN
-F 1 "GND" H 2150 4300 50  0000 C CNN
-F 2 "" H 2150 4450 50  0000 C CNN
-F 3 "" H 2150 4450 50  0000 C CNN
-	1    2150 4450
-	0    1    1    0
 $EndComp
 Wire Wire Line
@@
 	0    1    1    0
 $EndComp
+$Comp
+L +5V #PWR?
+U 1 1 58D840CD
+P 2150 4450
+F 0 "#PWR?" H 2150 4300 50  0001 C CNN
+F 1 "+5V" H 2150 4590 50  0000 C CNN
+F 2 "" H 2150 4450 50  0000 C CNN
+F 3 "" H 2150 4450 50  0000 C CNN
+	1    2150 4450
+	0    -1   -1   0
+$EndComp
 $EndSCHEMATC
